File: CSW_DoorTerminal_PowerAdapter.kicad_sch (KiCad schematic)
At the start: 4 parts, among them J1 USB_A, J2 S5B-PH-K-S, J3 Screw_Terminal_01x02, J4 Screw_Terminal_01x02

Commit message: finished pcb
Connections:
- net GND: now also J2.3, J2.4, J2.5, J4.1 (Pin_1)
- net Vee: now reaches J2.1
- net Vee: now also J2.2, J4.2 (Pin_2)
Changed lines of the file:
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@@
 	(paper "A4")
 	(junction
+		(at 123.19 66.04)
+		(diameter 0)
+		(color 0 0 0 0)
+	)
+	(junction
 		(at 50.8 72.39)
 		(diameter 0)
 		(color 0 0 0 0)
 	)
+	(junction
+		(at 123.19 63.5)
+		(diameter 0)
+		(color 0 0 0 0)
+	)
+	(junction
+		(at 123.19 58.42)
+		(diameter 0)
+		(color 0 0 0 0)
+	)
+	(wire
+		(pts
+			(xy 100.33 66.04) (xy 100.33 76.2)
+		)
+		(stroke
+			(width 0)
+			(type default)
+		)
+	)
+	(wire
+		(pts
+			(xy 123.19 60.96) (xy 123.19 63.5)
+		)
+		(stroke
+			(width 0)
+			(type default)
+		)
+	)
 	(wire
 		(pts
@@
 	(wire
 		(pts
+			(xy 123.19 58.42) (xy 127 58.42)
+		)
+		(stroke
+			(width 0)
+			(type default)
+		)
+	)
+	(wire
+		(pts
 			(xy 48.26 72.39) (xy 48.26 69.85)
 		)
@@
 	(wire
 		(pts
+			(xy 123.19 63.5) (xy 123.19 66.04)
+		)
+		(stroke
+			(width 0)
+			(type default)
+		)
+	)
+	(wire
+		(pts
 			(xy 68.58 54.61) (xy 68.58 76.2)
 		)
@@
 	(wire
 		(pts
+			(xy 127 63.5) (xy 123.19 63.5)
+		)
+		(stroke
+			(width 0)
+			(type default)
+		)
+	)
+	(wire
+		(pts
 			(xy 50.8 72.39) (xy 50.8 69.85)
 		)
@@
 	(wire
 		(pts
+			(xy 123.19 55.88) (xy 123.19 58.42)
+		)
+		(stroke
+			(width 0)
+			(type default)
+		)
+	)
+	(wire
+		(pts
 			(xy 60.96 62.23) (xy 60.96 59.69)
 		)
@@
 	(wire
 		(pts
+			(xy 123.19 66.04) (xy 127 66.04)
+		)
+		(stroke
+			(width 0)
+			(type default)
+		)
+	)
+	(wire
+		(pts
 			(xy 58.42 62.23) (xy 60.96 62.23)
 		)
@@
 	(wire
 		(pts
+			(xy 127 60.96) (xy 123.19 60.96)
+		)
+		(stroke
+			(width 0)
+			(type default)
+		)
+	)
+	(wire
+		(pts
+			(xy 97.79 76.2) (xy 97.79 58.42)
+		)
+		(stroke
+			(width 0)
+			(type default)
+		)
+	)
+	(wire
+		(pts
+			(xy 127 55.88) (xy 123.19 55.88)
+		)
+		(stroke
+			(width 0)
+			(type default)
+		)
+	)
+	(wire
+		(pts
 			(xy 50.8 72.39) (xy 48.26 72.39)
 		)
@@
 		(pts
 			(xy 68.58 54.61) (xy 58.42 54.61)
+		)
+		(stroke
+			(width 0)
+			(type default)
+		)
+	)
+	(wire
+		(pts
+			(xy 97.79 58.42) (xy 123.19 58.42)
+		)
+		(stroke
+			(width 0)
+			(type default)
+		)
+	)
+	(wire
+		(pts
+			(xy 100.33 66.04) (xy 123.19 66.04)
 		)
 		(stroke
@@
 		(effects
 			(font
+				(size 1.27 1.27)
+			)
+			(justify left bottom)
+		)
+	)
+	(label "Vee"
+		(at 113.03 58.42 0)
+		(effects
+			(font
+				(size 1.27 1.27)
+			)
+			(justify left bottom)
+		)
+	)
+	(label "GND"
+		(at 113.03 66.04 0)
+		(effects
+			(font

Commit message: added some metadata
Other:
- title: (none) -> Door Terminal Adapter PCB
Changed lines of the file:
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@@
 	(generator "eeschema")
 	(generator_version "10.0")
-	(paper "A4")
+	(paper "A5")
+	(title_block
+		(title "Door Terminal Adapter PCB")
+		(rev "V 1.0")
+	)
 	(junction
 		(at 123.19 66.04)
